Commit message: tool turned 90degrees

File: kuka_robot_bringup/robot/kr120toolv3.xacro (robot description, xacro)
@@ -6,15 +6,5 @@
     <kuka_kr120r2500pro prefix=""/>
     <gripper_6 parent="tool0" prefix="">
-		<origin xyz="0 0 0" rpy="0 0 0" />
+		<origin xyz="0 0 0" rpy="0 0 ${PI/2}" />
 	</gripper_6>
-    <!--link name="world"/>
-	<joint name="fixed" type="fixed">
-		<parent link="world"/>
-		<child link="base_link"/>
-	</joint>
-  <link name="base_link"/>
-  <gripper_6 parent="base_link" prefix="">
-	<origin xyz="0 0 0" rpy="0 0 0" />
-  </gripper_6-->
-  <!--ros_control/-->
 </robot>
